File: pedal-psu.kicad_pcb (KiCad board)
At the start: 2 copper layers, 100 x 100 mm, 76 parts, among them J1 Conn_01x01_Male, J2 Conn_01x01_Male, J3 Conn_01x02_Male, J4 Conn_01x02_Male, J5 Conn_01x02_Male, J6 Conn_01x02_Male, J7 Conn_01x02_Male, J8 Conn_01x02_Male, T1 Transformer_1P_1S, U1 LM78L09, U2 LM78L09, U3 LM78L09, U4 LM78L09, U5 LM7809_TO220, U6 LM317_3PinPackage, U7 LM358, U8 LM358, U9 LM358

Commit message: Machine version of PCB created.
Parts:
- added J9: Conn_01x10_Male, Connector_Molex:Molex_KK-254_AE-6410-10A_1x10_P2.54mm_Vertical, F.Cu at (127.3, 73.2)
- C1, C2, C3, C4: footprint Capacitor_THT:C_Radial_D10.0mm_H12.5mm_P5.00mm -> Capacitor_THT:CP_Radial_D10.0mm_P5.00mm_P7.50mm
- C11, C13, C17, C5, C7, C9: footprint Capacitor_THT:C_Radial_D6.3mm_H5.0mm_P2.50mm -> Capacitor_THT:CP_Radial_D6.3mm_P2.50mm
- R10, R11, R12, R13, R14, R15, R16, R17, R18, R19, R20, R3, R4, R5, R6, R7, R8, R9, U7, U8, U9: moved to F.Cu
- moved R6 48.0 mm to (94.0, 91.2), turned to 90 degrees
- moved R5 45.8 mm to (94.0, 96.5), turned to 90 degrees
- moved R19 41.8 mm to (138.2, 97.4), turned to 90 degrees
- moved R7 40.4 mm to (98.3, 87.7), turned to 0 degrees
- moved R16 36.5 mm to (99.9, 95.5)
- moved R13 31.0 mm to (131.6, 82.1), turned to 180 degrees
- moved R12 31.0 mm to (131.6, 87.7), turned to 0 degrees
- moved U7 30.1 mm to (131.8, 101.0), turned to 0 degrees
- moved R8 29.5 mm to (104.2, 87.7), turned to 0 degrees
- moved U9 28.1 mm to (104.3, 101.0), turned to 0 degrees
- moved R4 23.2 mm to (123.2, 106.2), turned to 270 degrees
- moved R11 22.1 mm to (126.6, 87.7), turned to 0 degrees
- moved R14 22.1 mm to (126.6, 82.1), turned to 180 degrees
- moved R20 20.8 mm to (126.8, 95.5)
- moved R15 18.5 mm to (109.5, 95.5)
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Routing:
- net +9V_5: track 161.2 -> 108.0 mm, vias 7 -> 4
- net Net-(J9-Pad6): track 3.55 -> 27.4 mm
- net Net-(J9-Pad1): track 4.77 -> 28.5 mm, vias 1 -> 0
- net Net-(J9-Pad5): track 3.56 -> 24.5 mm
- net Net-(J9-Pad4): track 3.56 -> 24.3 mm
- net Net-(J9-Pad2): track 3.54 -> 22.2 mm
- net Net-(J9-Pad3): track 3.56 -> 21.7 mm
- net +ADJV: track 61.5 -> 51.5 mm, vias 2 -> 1
- net +12V: track 190.9 -> 199.4 mm
- net V_SENSE: track 45.4 -> 40.9 mm
- net Net-(R11-Pad2): track 21.1 -> 17.8 mm
- net Net-(R10-Pad1): track 21.1 -> 17.8 mm
- net Net-(R10-Pad2): track 26.5 -> 23.2 mm
- net Net-(R8-Pad2): track 26.7 -> 23.4 mm
- net Net-(R12-Pad2): track 28.1 -> 24.8 mm
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- added copper zone on F.Cu, net GND
Other:
- net class Default: clearance 0.4 -> 0.2; trace_width 0.6 -> 0.25; via_dia 1.5 -> 0.8; via_drill 0.5 -> 0.4
- net class HighVoltage: via_dia 1.5 -> 0.8; via_drill 0.5 -> 0.4
- net class Power: clearance 0.4 -> 0.2; trace_width 1 -> 0.5; via_dia 1.5 -> 0.8; via_drill 0.5 -> 0.4
- rule trace_clearance: 0.4 -> 0.2
- board text added: "1"
- board text added: "2"
- board text added: "3"
- board text added: "4"
- board text added: "4.5-9V"
- board text added: "5"
- board text added: "6"
- board text added: "9V"
- board text added: "9V .5A"
- board text added: "GND"
- board text added: "SR pot"
- board text added: "Voltage pot"
- board text removed: "Pedal PSU"
